File: mouse1/mouse1-1/_restore_backup_2026-07-08T17-19-25-067/mouse1-1.kicad_sch (KiCad schematic)
At the start: 30 parts

Commit message: Made transparent LED, updated images in README
Parts:
- ENC1: footprint (none) -> AlpineRotaryEncoder:AlpineRotaryEncoder
